Commit message: deleted dynamixel-workbench submodule

File: mobilerobot_description/urdf/manipulator.urdf.xacro (robot description, xacro)
@@ -8,20 +8,4 @@
                                           joint6_lower_limit:=${-pi/2} joint6_upper_limit:=${pi/2}
                                           joint7_lower_limit:=${-pi/2} joint7_upper_limit:=${pi/2}">
-    <!--
-    <xacro:property name="joint1_lower_limit" value="${-pi/2}"/>
-    <xacro:property name="joint2_lower_limit" value="${-pi/2}"/>
-    <xacro:property name="joint3_lower_limit" value="${-pi/2}"/>
-    <xacro:property name="joint4_lower_limit" value="${-pi/2}"/>
-    <xacro:property name="joint5_lower_limit" value="${-pi/2}"/>
-    <xacro:property name="joint6_lower_limit" value="${-pi/2}"/>
-    <xacro:property name="joint7_lower_limit" value="${-pi/2}"/>
-    <xacro:property name="joint1_upper_limit" value="${pi/2}"/>
-    <xacro:property name="joint2_upper_limit" value="0"/>
-    <xacro:property name="joint3_upper_limit" value="${pi/2}"/>
-    <xacro:property name="joint4_upper_limit" value="${pi/2}"/>
-    <xacro:property name="joint5_upper_limit" value="${pi/2}"/>
-    <xacro:property name="joint6_upper_limit" value="${pi/2}"/>
-    <xacro:property name="joint7_upper_limit" value="${pi/2}"/>
-    -->
     <link name="${prefix}link1">
       <visual>

File: mobilerobot_description/urdf/mobile_chassis.transmission.xacro (robot description, xacro)
@@ -1,4 +1,3 @@
-<robot xmlns:xacro="http://wiki.ros.org/xacro"
-       name="mobilerobot" >
+<robot xmlns:xacro="http://wiki.ros.org/xacro">
   <xacro:macro name="mobile_chassis_transmission" params="prefix">
     <transmission name="${prefix}forward_left_joint_trans">
