Commit message: Add transmission to URDF

File: mobilerobot_description/urdf/mobile_chassis.transmission.xacro (robot description, xacro)
@@ -1,8 +1,8 @@
 <robot xmlns:xacro="http://wiki.ros.org/xacro">
-  <xacro:macro name="mobile_chassis_transmission" params="prefix">
+  <xacro:macro name="mobile_chassis_transmission" params="prefix hw_interface">
     <transmission name="${prefix}forward_left_joint_trans">
       <type>transmission_interface/SimpleTransmission</type>
       <joint name="forward_left_joint">
-        <hardwareInterface>hardware_interface/VelocityJointInterface</hardwareInterface>
+        <hardwareInterface>${hw_interface}</hardwareInterface>
       </joint>
       <actuator name="forward_left_actuator">
@@ -13,5 +13,5 @@
       <type>transmission_interface/SimpleTransmission</type>
       <joint name="forward_right_joint">
-        <hardwareInterface>hardware_interface/VelocityJointInterface</hardwareInterface>
+        <hardwareInterface>${hw_interface}</hardwareInterface>
       </joint>
       <actuator name="forward_right_actuator">
@@ -22,5 +22,5 @@
       <type>transmission_interface/SimpleTransmission</type>
       <joint name="backward_left_joint">
-        <hardwareInterface>hardware_interface/VelocityJointInterface</hardwareInterface>
+        <hardwareInterface>${hw_interface}</hardwareInterface>
       </joint>
       <actuator name="backward_left_actuator">
@@ -31,5 +31,5 @@
       <type>transmission_interface/SimpleTransmission</type>
       <joint name="backward_right_joint">
-        <hardwareInterface>hardware_interface/VelocityJointInterface</hardwareInterface>
+        <hardwareInterface>${hw_interface}</hardwareInterface>
       </joint>
       <actuator name="backward_right_actuator">

File: mobilerobot_description/urdf/mobile_chassis.urdf.xacro (robot description, xacro)
@@ -1,4 +1,5 @@
 <robot xmlns:xacro="http://wiki.ros.org/xacro">
-  <xacro:macro name="mobile_chassis" params="prefix">
+  <xacro:include filename="$(find mobilerobot_description)/urdf/mobile_chassis.transmission.xacro" />
+  <xacro:macro name="mobile_chassis" params="prefix transmission_hw_interface:=hardware_interface/VelocityActuatorInterface">
     <link name="${prefix}base_link">
       <visual>
@@ -67,4 +68,5 @@
         <geometry>
           <cylinder radius="0.075565" length="0.041"/>
+        </geometry>
         <material name="LightGrey">
           <color rgba="0.7 0.7 0.7 1.0"/>
@@ -124,4 +126,5 @@
       </collision>
     </link>
+    <xacro:mobile_chassis_transmission prefix="${prefix}" hw_interface="${transmission_hw_interface}"/>
   </xacro:macro>
 </robot>

Commit message: Modified transmission

File: mobilerobot_description/urdf/mobile_chassis.transmission.xacro (robot description, xacro)
@@ -7,4 +7,22 @@
       </joint>
       <actuator name="forward_left_actuator">
+        <mechanicalReduction>156</mechanicalReduction>
+      </actuator>
+    </transmission>
+    <transmission name="${prefix}backward_left_joint_trans">
+      <type>transmission_interface/SimpleTransmission</type>
+      <joint name="backward_left_joint">
+        <hardwareInterface>${hw_interface}</hardwareInterface>
+      </joint>
+      <actuator name="backward_left_actuator">
+        <mechanicalReduction>156</mechanicalReduction>
+      </actuator>
+    </transmission>
+    <transmission name="${prefix}backward_right_joint_trans">
+      <type>transmission_interface/SimpleTransmission</type>
+      <joint name="backward_right_joint">
+        <hardwareInterface>${hw_interface}</hardwareInterface>
+      </joint>
+      <actuator name="backward_right_actuator">
         <mechanicalReduction>156</mechanicalReduction>
       </actuator>
@@ -19,22 +37,4 @@
       </actuator>
     </transmission>
-    <transmission name="backward_left_joint_trans">
-      <type>transmission_interface/SimpleTransmission</type>
-      <joint name="backward_left_joint">
-        <hardwareInterface>${hw_interface}</hardwareInterface>
-      </joint>
-      <actuator name="backward_left_actuator">
-        <mechanicalReduction>156</mechanicalReduction>
-      </actuator>
-    </transmission>
-    <transmission name="backward_right_joint_trans">
-      <type>transmission_interface/SimpleTransmission</type>
-      <joint name="backward_right_joint">
-        <hardwareInterface>${hw_interface}</hardwareInterface>
-      </joint>
-      <actuator name="backward_right_actuator">
-        <mechanicalReduction>156</mechanicalReduction>
-      </actuator>
-    </transmission>
   </xacro:macro>
 </robot>
