Commit message: Modified URDF-Mecanum link geometry cylinder

File: mobilerobot_description/urdf/mobile_chassis.urdf.xacro (robot description, xacro)
@@ -38,7 +38,7 @@
       </visual>
       <collision>
-        <origin xyz="0 -0.13077 0" rpy="0 0 ${pi/2}"/>
+        <origin xyz="0 0 0" rpy="${pi/2} 0 0"/>
         <geometry>
-          <mesh filename="package://mobilerobot_description/meshes/mecanum_link.stl" scale="0.001 0.001 0.001"/>
+          <cylinder radius="0.075565" length="0.041"/>
         </geometry>
         <material name="LightGrey">
@@ -64,8 +64,7 @@
       </visual>
       <collision>
-        <origin xyz="0 0.13077 0" rpy="0 0 -${pi/2}"/>
+        <origin xyz="0 0 0" rpy="${pi/2} 0 0"/>
         <geometry>
-          <mesh filename="package://mobilerobot_description/meshes/mecanum_link.stl" scale="0.001 0.001 0.001"/>
-        </geometry>
+          <cylinder radius="0.075565" length="0.041"/>
         <material name="LightGrey">
           <color rgba="0.7 0.7 0.7 1.0"/>
@@ -90,7 +89,7 @@
       </visual>
       <collision>
-        <origin xyz="0 -0.13077 0" rpy="0 0 ${pi/2}"/>
+        <origin xyz="0 0 0" rpy="${pi/2} 0 0"/>
         <geometry>
-          <mesh filename="package://mobilerobot_description/meshes/mecanum_link.stl" scale="0.001 0.001 0.001"/>
+          <cylinder radius="0.075565" length="0.041"/>
         </geometry>
         <material name="LightGrey">
@@ -116,7 +115,7 @@
       </visual>
       <collision>
-        <origin xyz="0 0.13077 0" rpy="0 0 -${pi/2}"/>
+        <origin xyz="0 0 0" rpy="${pi/2} 0 0"/>
         <geometry>
-          <mesh filename="package://mobilerobot_description/meshes/mecanum_link.stl" scale="0.001 0.001 0.001"/>
+          <cylinder radius="0.075565" length="0.041"/>
         </geometry>
         <material name="LightGrey">

File: mobilerobot_description/urdf/mobilerobot.urdf (robot description, URDF)
Before this commit: robot mobilerobot, 15 links, 14 joints
Links:
- link backward_left_mecanum_link: geometry collision cylinder length=0.041 radius=0.075565; visual mesh filename=package://mobilerobot_description/meshes/mecanum_link.stl scale=0.001 0.001 0.001
- link backward_right_mecanum_link: geometry collision cylinder length=0.041 radius=0.075565; visual mesh filename=package://mobilerobot_description/meshes/mecanum_link.stl scale=0.001 0.001 0.001
- link forward_left_mecanum_link: geometry collision cylinder length=0.041 radius=0.075565; visual mesh filename=package://mobilerobot_description/meshes/mecanum_link.stl scale=0.001 0.001 0.001
- link forward_right_mecanum_link: geometry collision cylinder length=0.041 radius=0.075565; visual mesh filename=package://mobilerobot_description/meshes/mecanum_link.stl scale=0.001 0.001 0.001

Commit message: Modified transmission

File: mobilerobot_description/urdf/mobile_chassis.urdf.xacro (robot description, xacro)
@@ -1,5 +1,5 @@
 <robot xmlns:xacro="http://wiki.ros.org/xacro">
   <xacro:include filename="$(find mobilerobot_description)/urdf/mobile_chassis.transmission.xacro" />
-  <xacro:macro name="mobile_chassis" params="prefix transmission_hw_interface:=hardware_interface/VelocityActuatorInterface">
+  <xacro:macro name="mobile_chassis" params="prefix transmission_hw_interface:=hardware_interface/VelocityJointInterface">
     <link name="${prefix}base_link">
       <visual>

Commit message: Update

File: mobilerobot_description/urdf/mobile_chassis.urdf.xacro (robot description, xacro)
@@ -41,5 +41,5 @@
         <origin xyz="0 0 0" rpy="${pi/2} 0 0"/>
         <geometry>
-          <cylinder radius="0.075565" length="0.041"/>
+          <cylinder radius="0.0762" length="0.041"/>
         </geometry>
         <material name="LightGrey">
@@ -67,5 +67,5 @@
         <origin xyz="0 0 0" rpy="${pi/2} 0 0"/>
         <geometry>
-          <cylinder radius="0.075565" length="0.041"/>
+          <cylinder radius="0.0762" length="0.041"/>
         </geometry>
         <material name="LightGrey">
@@ -93,5 +93,5 @@
         <origin xyz="0 0 0" rpy="${pi/2} 0 0"/>
         <geometry>
-          <cylinder radius="0.075565" length="0.041"/>
+          <cylinder radius="0.0762" length="0.041"/>
         </geometry>
         <material name="LightGrey">
@@ -119,5 +119,5 @@
         <origin xyz="0 0 0" rpy="${pi/2} 0 0"/>
         <geometry>
-          <cylinder radius="0.075565" length="0.041"/>
+          <cylinder radius="0.0762" length="0.041"/>
         </geometry>
         <material name="LightGrey">
