Commit message: Add hokuyo link to URDF

File: mobilerobot_description/urdf/mobilerobot.urdf (robot description, URDF)
Before this commit: robot mobilerobot, 15 links, 14 joints
Links:
- added link hokuyo_link; visual mesh filename=package://mobilerobot_description/meshes/hokuyo_urg_04.stl scale=0.001 0.001 0.001
- added link odom
Joints:
- added joint hokuyo_fixed: type fixed, parent base_link, child hokuyo_link, origin xyz=0.373 0 0.005 rpy=0 0 0
- added joint odom_fixed: type fixed, parent hokuyo_link, child odom, origin xyz=-0.0192 -0.0192 0.065 rpy=0 0 0

File: mobilerobot_description/urdf/mobilerobot.urdf.xacro (robot description, xacro)
@@ -39,3 +39,25 @@
     <origin xyz="0.048 0 0.075" rpy="0 0 0"/>
   </joint>
+  <joint name="hokuyo_fixed" type="fixed">
+    <parent link="base_link"/>
+    <child link="hokuyo_link"/>
+    <origin xyz="0.373 0 0.005" rpy="0 0 0"/>
+  </joint>
+  <link name="hokuyo_link">
+    <visual>
+      <origin xyz="-0.0192 -0.0192 0" rpy="1.57079632679 0 1.57079632679"/>
+      <geometry>
+        <mesh filename="package://mobilerobot_description/meshes/hokuyo_urg_04.stl" scale="0.001 0.001 0.001"/>
+      </geometry>
+      <material name="LightGrey">
+        <color rgba="0.7 0.7 0.7 1.0"/>
+      </material>
+    </visual>
+  </link>
+  <joint name="odom_fixed" type="fixed">
+    <parent link="hokuyo_link"/>
+    <child link="odom"/>
+    <origin xyz="-0.0192 -0.0192 0.065" rpy="0 0 0"/>
+  </joint>
+  <link name="odom"/>
 </robot>

Commit message: Fixed TF Problem

File: mobilerobot_description/urdf/mobilerobot.urdf (robot description, URDF)
Before this commit: robot mobilerobot, 17 links, 16 joints
Links:
- removed link odom
- added link hokuyo_scan
Joints:
- joint odom_fixed: child odom -> hokuyo_scan

File: mobilerobot_description/urdf/mobilerobot.urdf.xacro (robot description, xacro)
@@ -57,7 +57,7 @@
   <joint name="odom_fixed" type="fixed">
     <parent link="hokuyo_link"/>
-    <child link="odom"/>
+    <child link="hokuyo_scan"/>
     <origin xyz="-0.0192 -0.0192 0.065" rpy="0 0 0"/>
   </joint>
-  <link name="odom"/>
+  <link name="hokuyo_scan"/>
 </robot>

Commit message: Modified  Link Name hokuyo_scan to laser_scan

File: mobilerobot_description/urdf/mobilerobot.urdf (robot description, URDF)
Before this commit: robot mobilerobot, 17 links, 16 joints
Links:
- removed link hokuyo_scan
- added link laser_scan
Joints:
- removed joint odom_fixed
- added joint laser_fixed: type fixed, parent hokuyo_link, child laser_scan, origin xyz=-0.0192 -0.0192 0.065 rpy=0 0 0

File: mobilerobot_description/urdf/mobilerobot.urdf.xacro (robot description, xacro)
@@ -55,9 +55,9 @@
     </visual>
   </link>
-  <joint name="odom_fixed" type="fixed">
+  <joint name="laser_fixed" type="fixed">
     <parent link="hokuyo_link"/>
-    <child link="hokuyo_scan"/>
+    <child link="laser_scan"/>
     <origin xyz="-0.0192 -0.0192 0.065" rpy="0 0 0"/>
   </joint>
-  <link name="hokuyo_scan"/>
+  <link name="laser_scan"/>
 </robot>

Commit message: Modified Manipulator joint4 upper limit

File: mobilerobot_description/urdf/mobilerobot.urdf (robot description, URDF)
Before this commit: robot mobilerobot, 17 links, 16 joints
Links:
- link backward_left_mecanum_link: geometry collision cylinder length=0.041 radius=0.0762; visual mesh filename=package://mobilerobot_description/meshes/mecanum_link.stl scale=0.001 0.001 0.001
- link backward_right_mecanum_link: geometry collision cylinder length=0.041 radius=0.0762; visual mesh filename=package://mobilerobot_description/meshes/mecanum_link.stl scale=0.001 0.001 0.001
- link forward_left_mecanum_link: geometry collision cylinder length=0.041 radius=0.0762; visual mesh filename=package://mobilerobot_description/meshes/mecanum_link.stl scale=0.001 0.001 0.001
- link forward_right_mecanum_link: geometry collision cylinder length=0.041 radius=0.0762; visual mesh filename=package://mobilerobot_description/meshes/mecanum_link.stl scale=0.001 0.001 0.001
Joints:
- joint joint4: limit lower=-1.57079632679 upper=1.57079632679 effort=1000 velocity=6.5 -> lower=0 upper=2.09439510239 effort=1000 velocity=6.5

File: mobilerobot_description/urdf/mobilerobot.urdf.xacro (robot description, xacro)
@@ -6,5 +6,5 @@
   <xacro:include filename="$(find mobilerobot_description)/urdf/ball_screw.transmission.xacro"/>
   <xacro:mobile_chassis prefix=""/>
-  <xacro:manipulator prefix="" joint2_upper_limit="0"/>
+  <xacro:manipulator prefix="" joint2_upper_limit="0" joint4_lower_limit="0" joint4_upper_limit="${2*pi/3}"/>
   <xacro:ball_screw_transmission prefix="" hw_interface="hardware_interface/PositionJointInterface"/>
   <xacro:property name="ball_screw_lower_limit" value="-0.77"/>

Commit message: Modified Model

File: mobilerobot_description/urdf/mobilerobot.urdf (robot description, URDF)
Before this commit: robot mobilerobot, 17 links, 16 joints
Links:
- added link zed_support; visual mesh filename=package://mobilerobot_description/meshes/zed_support.stl scale=0.001 0.001 0.001
Joints:
- added joint zed_support_fixed: type fixed, parent link7, child zed_support, origin xyz=0 0 0 rpy=0 0 0

File: mobilerobot_description/urdf/mobilerobot.urdf.xacro (robot description, xacro)
@@ -39,4 +39,20 @@
     <origin xyz="0.048 0 0.075" rpy="0 0 0"/>
   </joint>
+  <joint name="zed_support_fixed" type="fixed">
+    <parent link="link7"/>
+    <child link="zed_support"/>
+    <origin xyz="0 0 0" rpy="0 0 0"/>
+  </joint>
+  <link name="zed_support">
+    <visual>
+      <origin xyz="0 0 0" rpy="0 0 0"/>
+      <geometry>
+        <mesh filename="package://mobilerobot_description/meshes/zed_support.stl" scale="0.001 0.001 0.001"/>
+      </geometry>
+      <material name="LightGrey">
+        <color rgba="0.7 0.7 0.7 1.0"/>
+      </material>
+    </visual>
+  </link>
   <joint name="hokuyo_fixed" type="fixed">
     <parent link="base_link"/>

Commit message: add zed link

File: mobilerobot_description/urdf/mobilerobot.urdf (robot description, URDF)
Before this commit: robot mobilerobot, 18 links, 17 joints
Links:
- added link zed_camera_center; visual mesh filename=package://mobilerobot_description/meshes/ZED.stl
- added link zed_left_camera_frame
- added link zed_left_camera_optical_frame
- added link zed_right_camera_frame
- added link zed_right_camera_optical_frame
Joints:
- added joint zed_camera_center_joint: type fixed, parent zed_support, child zed_camera_center, origin xyz=0.034 0 0 rpy=0 1.57079632679 0
- added joint zed_left_camera_joint: type fixed, parent zed_camera_center, child zed_left_camera_frame, origin xyz=0 0.06 0 rpy=0 0 0
- added joint zed_left_camera_optical_joint: type fixed, parent zed_left_camera_frame, child zed_left_camera_optical_frame, origin xyz=0 0 0 rpy=-1.57079632679 0.0 -1.57079632679
- added joint zed_right_camera_joint: type fixed, parent zed_camera_center, child zed_right_camera_frame, origin xyz=0 -0.06 0 rpy=0 0 0
- added joint zed_right_camera_optical_joint: type fixed, parent zed_right_camera_frame, child zed_right_camera_optical_frame, origin xyz=0 0 0 rpy=-1.57079632679 0.0 -1.57079632679
- joint zed_support_fixed: origin xyz=0 0 0 rpy=0 0 0 -> xyz=0.021 -0.045 -0.075 rpy=0 0 0

File: mobilerobot_description/urdf/mobilerobot.urdf.xacro (robot description, xacro)
@@ -42,9 +42,9 @@
     <parent link="link7"/>
     <child link="zed_support"/>
-    <origin xyz="0 0 0" rpy="0 0 0"/>
+    <origin xyz="0.021 -0.045 -0.075" rpy="0 0 0"/>
   </joint>
   <link name="zed_support">
     <visual>
-      <origin xyz="0 0 0" rpy="0 0 0"/>
+      <origin xyz="0 0 0" rpy="-${pi/2} 0 -${pi/2}"/>
       <geometry>
         <mesh filename="package://mobilerobot_description/meshes/zed_support.stl" scale="0.001 0.001 0.001"/>
@@ -55,4 +55,46 @@
     </visual>
   </link>
+  <joint name="zed_camera_center_joint" type="fixed">
+    <parent link="zed_support"/>
+    <child link="zed_camera_center"/>
+    <origin xyz="0.034 0 0" rpy="0 ${pi/2} 0"/>
+  </joint>
+  <link name="zed_camera_center">
+    <visual>
+      <origin xyz="0 0 0" rpy="0 0 0"/>
+      <geometry>
+        <mesh filename="package://mobilerobot_description/meshes/ZED.stl"/>
+      </geometry>
+      <material name="light_grey">
+        <color rgba="0.8 0.8 0.8 0.8"/>
+      </material>
+    </visual>
+  </link>
+<!-- Left Camera -->
+  <joint name="zed_left_camera_joint" type="fixed">
+      <parent link="zed_camera_center"/>
+      <child link="zed_left_camera_frame"/>
+      <origin xyz="0 0.06 0" rpy="0 0 0" />
+  </joint>
+  <link name="zed_left_camera_frame" />
+  <joint name="zed_left_camera_optical_joint" type="fixed">
+      <origin xyz="0 0 0" rpy="-1.57079632679 0.0 -1.57079632679"/>
+      <parent link="zed_left_camera_frame"/>
+      <child link="zed_left_camera_optical_frame"/>
+  </joint>
+  <link name="zed_left_camera_optical_frame"/>
+<!-- Right Camera -->
+  <joint name="zed_right_camera_joint" type="fixed">
+      <parent link="zed_camera_center"/>
+      <child link="zed_right_camera_frame"/>
+      <origin xyz="0 -0.06 0" rpy="0 0 0" />
+  </joint>
+  <link name="zed_right_camera_frame" />
+  <joint name="zed_right_camera_optical_joint" type="fixed">
+      <origin xyz="0 0 0" rpy="-1.57079632679 0.0 -1.57079632679"/>
+      <parent link="zed_right_camera_frame"/>
+      <child link="zed_right_camera_optical_frame"/>
+  </joint>
+  <link name="zed_right_camera_optical_frame"/>
   <joint name="hokuyo_fixed" type="fixed">
     <parent link="base_link"/>
